Commit message: added vesc_right ros2 control interface

File: vesc_hw_interface/launch/velocity_duty_test.ros2_control.xacro (robot description, xacro)
@@ -1,5 +1,5 @@
 <?xml version="1.0" encoding="UTF-8"?>
 <robot xmlns:xacro="http://www.ros.org/wiki/xacro">
-  <ros2_control name="vesc" type="actuator">
+  <ros2_control name="vesc_left" type="actuator">
     <hardware>
       <plugin>vesc_hw_interface/VescHwInterface</plugin>
@@ -55,3 +55,57 @@
     </joint>
   </ros2_control>
+  <ros2_control name="vesc_right" type="actuator">
+    <hardware>
+      <plugin>vesc_hw_interface/VescHwInterface</plugin>
+      <param name="port">/dev/ttyACM1</param>
+      <param name="gear_ratio">0.230769</param>
+      <param name="torque_const">1.0</param>
+      <param name="num_hall_sensors">3</param>
+      <param name="screw_lead">1.0</param>
+      <param name="num_rotor_poles">14</param>
+      <param name="servo/Kp">0.005</param>
+      <param name="servo/Ki">0.005</param>
+      <param name="servo/Kd">0.0025</param>
+      <param name="servo/i_clamp">1.0</param>
+      <param name="servo/duty_limiter">1.0</param>
+      <param name="servo/antiwindup">true</param>
+      <param name="servo/control_rate">100.0</param>
+      <param name="servo/calibration_current">6.0</param>
+      <param name="servo/calibration_duty">0.1</param>
+      <param name="servo/calibration_mode">current</param>
+      <param name="servo/calibration_position">0.0</param>
+      <param name="servo/enable_smooth_diff">true</param>
+      <param name="servo/smooth_diff/max_sample_sec">1.0</param>
+      <param name="servo/smooth_diff/max_smooth_step">10</param>
+      <param name="motor/Kp">0.1</param>
+      <param name="motor/Ki">0.01</param>
+      <param name="motor/Kd">0.02</param>
+      <param name="motor/i_clamp">1.0</param>
+      <param name="motor/duty_limiter">1.0</param>
+      <param name="motor/antiwindup">true</param>
+      <param name="motor/control_rate">100.0</param>
+      <param name="motor/enable_smooth_diff">true</param>
+      <param name="motor/smooth_diff/max_sample_sec">0.2</param>
+      <param name="motor/smooth_diff/max_smooth_step">10</param>
+      <param name="command_mode">velocity_duty</param>
+      <param name="joint_type">continuous</param>
+    </hardware>
+    <joint name="vesc_joint_right">
+      <command_interface name="position">
+        <param name="min">-1</param>
+        <param name="max">1</param>
+      </command_interface>
+      <command_interface name="velocity">
+        <param name="min">-1</param>
+        <param name="max">1</param>
+      </command_interface>
+      <command_interface name="effort">
+        <param name="min">-1</param>
+        <param name="max">1</param>
+      </command_interface>
+      <state_interface name="position"/>
+      <state_interface name="velocity"/>
+      <state_interface name="effort"/>
+    </joint>
+  </ros2_control>
 </robot>

Commit message: changing to diff drive controller

File: vesc_hw_interface/launch/velocity_duty_test.ros2_control.xacro (robot description, xacro)
@@ -1,5 +1,5 @@
 <?xml version="1.0" encoding="UTF-8"?>
 <robot xmlns:xacro="http://www.ros.org/wiki/xacro">
-  <ros2_control name="vesc" type="actuator">
+  <ros2_control name="vesc_left" type="actuator">
     <hardware>
       <plugin>vesc_hw_interface/VescHwInterface</plugin>
@@ -37,17 +37,71 @@
       <param name="joint_type">continuous</param>
     </hardware>
-    <joint name="vesc_joint">
-      <command_interface name="position">
+    <joint name="left_wheel_joint">
+      <!--<command_interface name="position">
         <param name="min">-1</param>
         <param name="max">1</param>
-      </command_interface>
+      </command_interface>!-->
       <command_interface name="velocity">
         <param name="min">-1</param>
         <param name="max">1</param>
       </command_interface>
-      <command_interface name="effort">
+      <!--<command_interface name="effort">
+        <param name="min">-1</param>
+        <param name="max">1</param>
+      </command_interface>!-->
+      <state_interface name="position"/>
+      <state_interface name="velocity"/>
+      <state_interface name="effort"/>
+    </joint>
+  </ros2_control>
+  <ros2_control name="vesc_right" type="actuator">
+    <hardware>
+      <plugin>vesc_hw_interface/VescHwInterface</plugin>
+      <param name="port">/dev/ttyACM1</param>
+      <param name="gear_ratio">0.25</param>
+      <param name="torque_const">1.0</param>
+      <param name="num_hall_sensors">1</param>
+      <param name="screw_lead">1.0</param>
+      <param name="num_rotor_poles">14</param>
+      <param name="servo/Kp">0.005</param>
+      <param name="servo/Ki">0.005</param>
+      <param name="servo/Kd">0.0025</param>
+      <param name="servo/i_clamp">1.0</param>
+      <param name="servo/duty_limiter">1.0</param>
+      <param name="servo/antiwindup">true</param>
+      <param name="servo/control_rate">100.0</param>
+      <param name="servo/calibration_current">6.0</param>
+      <param name="servo/calibration_duty">0.1</param>
+      <param name="servo/calibration_mode">current</param>
+      <param name="servo/calibration_position">0.0</param>
+      <param name="servo/enable_smooth_diff">true</param>
+      <param name="servo/smooth_diff/max_sample_sec">1.0</param>
+      <param name="servo/smooth_diff/max_smooth_step">10</param>
+      <param name="motor/Kp">0.1</param>
+      <param name="motor/Ki">0.01</param>
+      <param name="motor/Kd">0.02</param>
+      <param name="motor/i_clamp">1.0</param>
+      <param name="motor/duty_limiter">1.0</param>
+      <param name="motor/antiwindup">true</param>
+      <param name="motor/control_rate">100.0</param>
+      <param name="motor/enable_smooth_diff">true</param>
+      <param name="motor/smooth_diff/max_sample_sec">0.2</param>
+      <param name="motor/smooth_diff/max_smooth_step">10</param>
+      <param name="command_mode">velocity_duty</param>
+      <param name="joint_type">continuous</param>
+    </hardware>
+    <joint name="right_wheel_joint">
+      <!--<command_interface name="position">
+        <param name="min">-1</param>
+        <param name="max">1</param>
+      </command_interface>!-->
+      <command_interface name="velocity">
         <param name="min">-1</param>
         <param name="max">1</param>
       </command_interface>
+      <!--<command_interface name="effort">
+        <param name="min">-1</param>
+        <param name="max">1</param>
+      </command_interface>!-->
       <state_interface name="position"/>
       <state_interface name="velocity"/>
