Commit message: added base link

File: vesc-ros2/vesc_driver/description/robot_core.xacro (robot description, xacro)
@@ -30,4 +30,7 @@
         <color rgba="1 0 0 1"/>
     </material>
+    <!-- BASE LINK -->
+    <link name="base_link">
+    </link>
     <!-- CHASSIS LINK -->
     <joint name="chassis_joint" type="fixed">

Commit message: fixing measurements for desc

File: vesc-ros2/vesc_driver/description/robot_core.xacro (robot description, xacro)
@@ -1,17 +1,18 @@
 <?xml version="1.0"?>
 <robot xmlns:xacro="http://www.ros.org/wiki/xacro" >
-    <xacro:property name="chassis_length" value="0.335"/>
-    <xacro:property name="chassis_width" value="0.265"/>
-    <xacro:property name="chassis_height" value="0.138"/>
+    <xacro:property name="chassis_length" value="0.699"/>
+    <xacro:property name="chassis_width" value="0.406"/>
+    <xacro:property name="chassis_height" value="0.076"/>
     <xacro:property name="chassis_mass" value="1.0"/>
-    <xacro:property name="wheel_radius" value="0.033"/>
-    <xacro:property name="wheel_thickness" value="0.026"/>
+    <xacro:property name="wheel_radius" value="0.150"/>
+    <xacro:property name="wheel_thickness" value="0.045"/>
     <xacro:property name="wheel_mass" value="0.05"/>
-    <xacro:property name="wheel_offset_x" value="0.226"/>
-    <xacro:property name="wheel_offset_y" value="0.1485"/>
-    <xacro:property name="wheel_offset_z" value="0.01"/>
-    <xacro:property name="caster_wheel_radius" value="0.01"/>
+    <xacro:property name="wheel_offset_x" value="0.152"/>
+    <xacro:property name="wheel_offset_y" value="0.0"/>
+    <xacro:property name="wheel_offset_z" value="0.089"/>
+    <xacro:property name="caster_wheel_radius" value="0.100"/>
     <xacro:property name="caster_wheel_mass" value="0.01"/>
-    <xacro:property name="caster_wheel_offset_x" value="0.075"/>
+    <xacro:property name="caster_wheel_offset_x" value="0.0"/>
+    <xacro:property name="caster_wheel_offset_y" value="0.349"/>
     <xacro:property name="caster_wheel_offset_z" value="${wheel_offset_z - wheel_radius + caster_wheel_radius}"/>
     <material name="white">
@@ -55,5 +56,5 @@
     </link>
     <!-- LEFT WHEEL LINK -->
-    <joint name="left_wheel_joint" type="continuous">
+    <joint name="left_wheel_joint" type="fixed">
         <parent link="base_link"/>
         <child link="left_wheel"/>
@@ -75,5 +76,5 @@
     </link>
     <!-- RIGHT WHEEL LINK -->
-    <joint name="right_wheel_joint" type="continuous">
+    <joint name="right_wheel_joint" type="fixed">
         <parent link="base_link"/>
         <child link="right_wheel"/>

Commit message: desc

File: vesc-ros2/vesc_driver/description/robot_core.xacro (robot description, xacro)
@@ -38,5 +38,5 @@
         <parent link="base_link"/>
         <child link="chassis"/>
-        <origin xyz="${-wheel_offset_x} 0 ${-wheel_offset_z}"/>
+        <origin xyz="0 0 ${-wheel_offset_z}"/>
     </joint>
     <link name="chassis">

Commit message: desc

File: vesc-ros2/vesc_driver/description/robot_core.xacro (robot description, xacro)
@@ -38,9 +38,9 @@
         <parent link="base_link"/>
         <child link="chassis"/>
-        <origin xyz="0 0 ${-wheel_offset_z}"/>
+        <origin xyz="${-wheel_offset_x} 0 ${-wheel_offset_z}"/>
     </joint>
     <link name="chassis">
         <visual>
-            <origin xyz="${chassis_length/2} 0 ${chassis_height/2}"/>
+            <origin xyz="${chassis_length/2} 0 0.216"/>
             <geometry>
                 <box size="${chassis_length} ${chassis_width} ${chassis_height}"/>

Commit message: desc

File: vesc-ros2/vesc_driver/description/robot_core.xacro (robot description, xacro)
@@ -5,5 +5,5 @@
     <xacro:property name="chassis_height" value="0.076"/>
     <xacro:property name="chassis_mass" value="1.0"/>
-    <xacro:property name="wheel_radius" value="0.150"/>
+    <xacro:property name="wheel_radius" value="0.075"/>
     <xacro:property name="wheel_thickness" value="0.045"/>
     <xacro:property name="wheel_mass" value="0.05"/>
@@ -38,5 +38,5 @@
         <parent link="base_link"/>
         <child link="chassis"/>
-        <origin xyz="${-wheel_offset_x} 0 ${-wheel_offset_z}"/>
+        <origin xyz="${chassis_length/2} 0 ${-wheel_offset_z}"/>
     </joint>
     <link name="chassis">

Commit message: desc

File: vesc-ros2/vesc_driver/description/robot_core.xacro (robot description, xacro)
@@ -8,6 +8,6 @@
     <xacro:property name="wheel_thickness" value="0.045"/>
     <xacro:property name="wheel_mass" value="0.05"/>
-    <xacro:property name="wheel_offset_x" value="0.152"/>
-    <xacro:property name="wheel_offset_y" value="0.0"/>
+    <xacro:property name="wheel_offset_x" value="0.0"/>
+    <xacro:property name="wheel_offset_y" value="0.152"/>
     <xacro:property name="wheel_offset_z" value="0.089"/>
     <xacro:property name="caster_wheel_radius" value="0.100"/>
@@ -38,5 +38,5 @@
         <parent link="base_link"/>
         <child link="chassis"/>
-        <origin xyz="${chassis_length/2} 0 ${-wheel_offset_z}"/>
+        <origin xyz="${-chassis_length/2} 0 ${-wheel_offset_z}"/>
     </joint>
     <link name="chassis">

Commit message: desc

File: vesc-ros2/vesc_driver/description/robot_core.xacro (robot description, xacro)
@@ -13,6 +13,6 @@
     <xacro:property name="caster_wheel_radius" value="0.100"/>
     <xacro:property name="caster_wheel_mass" value="0.01"/>
-    <xacro:property name="caster_wheel_offset_x" value="0.0"/>
-    <xacro:property name="caster_wheel_offset_y" value="0.349"/>
+    <xacro:property name="caster_wheel_offset_x" value="0.349"/>
+    <xacro:property name="caster_wheel_offset_y" value="0.0"/>
     <xacro:property name="caster_wheel_offset_z" value="${wheel_offset_z - wheel_radius + caster_wheel_radius}"/>
     <material name="white">
@@ -38,9 +38,9 @@
         <parent link="base_link"/>
         <child link="chassis"/>
-        <origin xyz="${-chassis_length/2} 0 ${-wheel_offset_z}"/>
+        <origin xyz="{-wheel_offset_x} 0 ${-wheel_offset_z}"/>
     </joint>
     <link name="chassis">
         <visual>
-            <origin xyz="${chassis_length/2} 0 0.216"/>
+            <origin xyz="0 0 0"/>
             <geometry>
                 <box size="${chassis_length} ${chassis_width} ${chassis_height}"/>

Commit message: desc

File: vesc-ros2/vesc_driver/description/robot_core.xacro (robot description, xacro)
@@ -38,5 +38,5 @@
         <parent link="base_link"/>
         <child link="chassis"/>
-        <origin xyz="{-wheel_offset_x} 0 ${-wheel_offset_z}"/>
+        <origin xyz="0 0 .216"/>
     </joint>
     <link name="chassis">

Commit message: desc

File: vesc-ros2/vesc_driver/description/robot_core.xacro (robot description, xacro)
@@ -38,9 +38,9 @@
         <parent link="base_link"/>
         <child link="chassis"/>
-        <origin xyz="0 0 .216"/>
+        <origin xyz="0 0 0"/>
     </joint>
     <link name="chassis">
         <visual>
-            <origin xyz="0 0 0"/>
+            <origin xyz="0 0 .216>
             <geometry>
                 <box size="${chassis_length} ${chassis_width} ${chassis_height}"/>

Commit message: desc

File: vesc-ros2/vesc_driver/description/robot_core.xacro (robot description, xacro)
@@ -42,5 +42,5 @@
     <link name="chassis">
         <visual>
-            <origin xyz="0 0 .216>
+            <origin xyz="0 0 .216">
             <geometry>
                 <box size="${chassis_length} ${chassis_width} ${chassis_height}"/>

Commit message: desc

File: vesc-ros2/vesc_driver/description/robot_core.xacro (robot description, xacro)
@@ -42,5 +42,5 @@
     <link name="chassis">
         <visual>
-            <origin xyz="0 0 .216">
+            <origin xyz="0 0 0.216">
             <geometry>
                 <box size="${chassis_length} ${chassis_width} ${chassis_height}"/>

Commit message: desc

File: vesc-ros2/vesc_driver/description/robot_core.xacro (robot description, xacro)
@@ -42,5 +42,5 @@
     <link name="chassis">
         <visual>
-            <origin xyz="0 0 0.216">
+            <origin xyz="0 0 .216"/>
             <geometry>
                 <box size="${chassis_length} ${chassis_width} ${chassis_height}"/>

Commit message: desc

File: vesc-ros2/vesc_driver/description/robot_core.xacro (robot description, xacro)
@@ -59,5 +59,5 @@
         <parent link="base_link"/>
         <child link="left_wheel"/>
-        <origin xyz="0 ${wheel_offset_y} 0" rpy="-${pi/2} 0 0" />
+        <origin xyz="0 ${wheel_offset_y} ${wheel_radius/2}" rpy="-${pi/2} 0 0" />
         <axis xyz="0 0 1"/>
     </joint>

Commit message: desc

File: vesc-ros2/vesc_driver/description/robot_core.xacro (robot description, xacro)
@@ -42,5 +42,5 @@
     <link name="chassis">
         <visual>
-            <origin xyz="0 0 .216"/>
+            <origin xyz="0 0 .140"/>
             <geometry>
                 <box size="${chassis_length} ${chassis_width} ${chassis_height}"/>
@@ -59,5 +59,5 @@
         <parent link="base_link"/>
         <child link="left_wheel"/>
-        <origin xyz="0 ${wheel_offset_y} ${wheel_radius/2}" rpy="-${pi/2} 0 0" />
+        <origin xyz="0 ${wheel_offset_y} 0" rpy="-${pi/2} 0 0" />
         <axis xyz="0 0 1"/>
     </joint>

Commit message: desc

File: vesc-ros2/vesc_driver/description/robot_core.xacro (robot description, xacro)
@@ -13,7 +13,7 @@
     <xacro:property name="caster_wheel_radius" value="0.100"/>
     <xacro:property name="caster_wheel_mass" value="0.01"/>
-    <xacro:property name="caster_wheel_offset_x" value="0.349"/>
+    <xacro:property name="caster_wheel_offset_x" value="0.100"/>
     <xacro:property name="caster_wheel_offset_y" value="0.0"/>
-    <xacro:property name="caster_wheel_offset_z" value="${wheel_offset_z - wheel_radius + caster_wheel_radius}"/>
+    <xacro:property name="caster_wheel_offset_z" value=".089"/>
     <material name="white">
         <color rgba="1 1 1 1" />

Commit message: desc

File: vesc-ros2/vesc_driver/description/robot_core.xacro (robot description, xacro)
@@ -96,15 +96,16 @@
     </link>
     <!-- CASTER WHEEL LINK -->
-    <joint name="caster_wheel_joint" type="fixed">
-        <parent link="chassis"/>
-        <child link="caster_wheel"/>
-        <origin xyz="${caster_wheel_offset_x} 0 ${caster_wheel_offset_z}"/>
+    <joint name="fcaster_wheel_joint" type="fixed">
+        <parent link="base_link"/>
+        <child link="fcaster_wheel"/>
+        <origin xyz="0 ${caster_offset_y} 0" rpy="${pi/2} 0 0" />
+        <axis xyz="0 0 -1"/>
     </joint>
-    <link name="caster_wheel">
+    <link name="fcaster_wheel">
         <visual>
             <geometry>
-                <sphere radius="${caster_wheel_radius}"/>
+                <cylinder radius="${caster_wheel_radius}" length="${wheel_thickness}"/>
             </geometry>
-            <material name="white"/>
+            <material name="blue"/>
         </visual>
         <collision>

Commit message: desc

File: vesc-ros2/vesc_driver/description/robot_core.xacro (robot description, xacro)
@@ -99,5 +99,5 @@
         <parent link="base_link"/>
         <child link="fcaster_wheel"/>
-        <origin xyz="0 ${caster_offset_y} 0" rpy="${pi/2} 0 0" />
+        <origin xyz="0 ${caster_wheel_offset_y} 0" rpy="${pi/2} 0 0" />
         <axis xyz="0 0 -1"/>
     </joint>

Commit message: desc

File: vesc-ros2/vesc_driver/description/robot_core.xacro (robot description, xacro)
@@ -11,5 +11,5 @@
     <xacro:property name="wheel_offset_y" value="0.152"/>
     <xacro:property name="wheel_offset_z" value="0.089"/>
-    <xacro:property name="caster_wheel_radius" value="0.100"/>
+    <xacro:property name="caster_wheel_radius" value="0.075"/>
     <xacro:property name="caster_wheel_mass" value="0.01"/>
     <xacro:property name="caster_wheel_offset_x" value="0.100"/>
@@ -99,5 +99,5 @@
         <parent link="base_link"/>
         <child link="fcaster_wheel"/>
-        <origin xyz="0 ${caster_wheel_offset_y} 0" rpy="${pi/2} 0 0" />
+        <origin xyz="${caster_wheel_offset_x} 0 0" rpy="${pi/2} 0 0" />
         <axis xyz="0 0 -1"/>
     </joint>

Commit message: desc

File: vesc-ros2/vesc_driver/description/robot_core.xacro (robot description, xacro)
@@ -1,5 +1,5 @@
 <?xml version="1.0"?>
 <robot xmlns:xacro="http://www.ros.org/wiki/xacro" >
-    <xacro:property name="chassis_length" value="0.699"/>
+    <xacro:property name="chassis_length" value="0.508"/>
     <xacro:property name="chassis_width" value="0.406"/>
     <xacro:property name="chassis_height" value="0.076"/>

Commit message: desc

File: vesc-ros2/vesc_driver/description/robot_core.xacro (robot description, xacro)
@@ -13,5 +13,5 @@
     <xacro:property name="caster_wheel_radius" value="0.075"/>
     <xacro:property name="caster_wheel_mass" value="0.01"/>
-    <xacro:property name="caster_wheel_offset_x" value="0.100"/>
+    <xacro:property name="caster_wheel_offset_x" value="0.150"/>
     <xacro:property name="caster_wheel_offset_y" value="0.0"/>
     <xacro:property name="caster_wheel_offset_z" value=".089"/>
@@ -115,3 +115,23 @@
         </collision>
     </link>
+    <!-- CASTER WHEEL LINK -->
+    <joint name="rcaster_wheel_joint" type="fixed">
+        <parent link="base_link"/>
+        <child link="rcaster_wheel"/>
+        <origin xyz="${-caster_wheel_offset_x} 0 0" rpy="${pi/2} 0 0" />
+        <axis xyz="0 0 -1"/>
+    </joint>
+    <link name="rcaster_wheel">
+        <visual>
+            <geometry>
+                <cylinder radius="${caster_wheel_radius}" length="${wheel_thickness}"/>
+            </geometry>
+            <material name="blue"/>
+        </visual>
+        <collision>
+            <geometry>
+                <sphere radius="${caster_wheel_radius}"/>
+            </geometry>
+        </collision>
+    </link>
 </robot>
